File: hardware/kicad/forest-rover.kicad_pcb (KiCad board)
At the start: 4 copper layers, 100 x 80 mm, 0 parts

Commit message: Refine repo wording and KiCad scaffolding
Other:
- board text added: "100 mm x 80 mm board outline"
- board text added: "Analog Front-End"
- board text added: "CM4 / External I O"
- board text added: "DRV8871 x2, stitching vias, local bulk caps"
- board text added: "Ground stitching fence along motor section boundary"
- board text added: "Keep switching regulators away from analog front-end"
- board text added: "MCU Core"
- board text added: "Motor Driver Zone"
- board text added: "PIR conditioning and thermistor ADC path"
- board text added: "Power Stage"
- board text added: "RF Edge Section"
- board text added: "RFM95W, PI match, SMA edge connector"
- board text added: "Reserve uninterrupted reference under MCU and RF traces on In1.Cu"
- board text added: "STM32F407, flash, crystals, SWD"
- board text added: "Solar input, charger, 5V buck, 3.3V LDO"
- board text added: "Split In2.Cu into VBAT / +5V / +3V3 islands with controlled return paths"
- board text added: "UART, I2C, USB-C, JST sensor headers"
- board text removed: "4-layer placeholder layout scaffold"
- board text removed: "Analog sensor front-end isolated in lower-left quadrant"
- board text removed: "Buck + solar charger floorplan on left edge"
- board text removed: "Keep RF section on right board edge"
- board text removed: "Motor driver zone with stitching vias along lower edge"
Changed lines of the file:
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@@
     (title "Forest Surveillance Rover Main Controller PCB")
     (company "Team Onyx India")
-    (rev "A"))
+    (rev "A")
+    (comment 1 "Layout floorplan with named nets")
+    (comment 2 "Board target approximately 100mm x 80mm"))
   (layers
     (0 "F.Cu" signal)
@@
   (setup
     (pad_to_mask_clearance 0)
+    (stackup
+      (layer "F.Cu" (type "copper") (thickness 0.035))
+      (layer "dielectric 1" (type "prepreg") (thickness 0.18) (material "FR4"))
+      (layer "In1.Cu" (type "copper") (thickness 0.035))
+      (layer "dielectric 2" (type "core") (thickness 1.10) (material "FR4"))
+      (layer "In2.Cu" (type "copper") (thickness 0.035))
+      (layer "dielectric 3" (type "prepreg") (thickness 0.18) (material "FR4"))
+      (layer "B.Cu" (type "copper") (thickness 0.035))
+      (copper_finish "ENIG")
+      (dielectric_constraints yes))
     (pcbplotparams
       (layerselection 0x00010fc_ffffffff)
       (plot_on_all_layers_selection 0x0000000_00000000)
       (disableapertmacros false)))
+  (property "StackupIntent" "Signal-GND-Power-Signal")
+  (property "LayoutStatus" "Preliminary floorplan")
   (net 0 "")
+  (net 1 "VBAT")
+  (net 2 "+5V")
+  (net 3 "+3V3")
+  (net 4 "MOTOR_VBAT")
+  (net 5 "GND")
+  (net 6 "I2C1_SCL")
+  (net 7 "I2C1_SDA")
+  (net 8 "LORA_SPI_SCK")
+  (net 9 "LORA_SPI_MOSI")
+  (net 10 "LORA_SPI_MISO")
+  (net 11 "CM4_UART_TX")
+  (net 12 "CM4_UART_RX")
   (gr_rect (start 0 0) (end 100 80) (layer "Edge.Cuts") (width 0.1) (fill none))
-  (gr_text "Forest Rover Rev A" (at 10 10) (layer "F.SilkS"))
-  (gr_text "4-layer placeholder layout scaffold" (at 10 14) (layer "F.SilkS"))
-  (gr_text "Keep RF section on right board edge" (at 64 10) (layer "Dwgs.User"))
-  (gr_text "Buck + solar charger floorplan on left edge" (at 8 22) (layer "Dwgs.User"))
-  (gr_text "Analog sensor front-end isolated in lower-left quadrant" (at 8 66) (layer "Dwgs.User"))
-  (gr_text "Motor driver zone with stitching vias along lower edge" (at 48 68) (layer "Dwgs.User"))
+  (gr_rect (start 6 8) (end 28 32) (layer "Dwgs.User") (width 0.15) (fill none))
+  (gr_rect (start 31 8) (end 62 42) (layer "Dwgs.User") (width 0.15) (fill none))
+  (gr_rect (start 66 8) (end 94 25) (layer "Dwgs.User") (width 0.15) (fill none))
+  (gr_rect (start 7 48) (end 31 72) (layer "Dwgs.User") (width 0.15) (fill none))
+  (gr_rect (start 39 49) (end 76 73) (layer "Dwgs.User") (width 0.15) (fill none))
+  (gr_rect (start 79 45) (end 94 67) (layer "Dwgs.User") (width 0.15) (fill none))
+  (gr_text "Forest Rover Rev A" (at 9 9) (layer "F.SilkS"))
+  (gr_text "100 mm x 80 mm board outline" (at 9 13) (layer "F.SilkS"))
+  (gr_text "Power Stage" (at 11 12) (layer "Dwgs.User"))
+  (gr_text "Solar input, charger, 5V buck, 3.3V LDO" (at 8 17) (layer "Dwgs.User"))
+  (gr_text "MCU Core" (at 42 12) (layer "Dwgs.User"))
+  (gr_text "STM32F407, flash, crystals, SWD" (at 34 17) (layer "Dwgs.User"))
+  (gr_text "RF Edge Section" (at 70 12) (layer "Dwgs.User"))
+  (gr_text "RFM95W, PI match, SMA edge connector" (at 67 17) (layer "Dwgs.User"))
+  (gr_text "Analog Front-End" (at 10 53) (layer "Dwgs.User"))
+  (gr_text "PIR conditioning and thermistor ADC path" (at 8 58) (layer "Dwgs.User"))
+  (gr_text "Motor Driver Zone" (at 47 54) (layer "Dwgs.User"))
+  (gr_text "DRV8871 x2, stitching vias, local bulk caps" (at 41 59) (layer "Dwgs.User"))
+  (gr_text "CM4 / External I O" (at 80 50) (layer "Dwgs.User"))
+  (gr_text "UART, I2C, USB-C, JST sensor headers" (at 79 55) (layer "Dwgs.User"))
+  (gr_text "Keep switching regulators away from analog front-end" (at 6 39) (layer "Cmts.User"))
+  (gr_text "Reserve uninterrupted reference under MCU and RF traces on In1.Cu" (at 32 45) (layer "Cmts.User"))
+  (gr_text "Split In2.Cu into VBAT / +5V / +3V3 islands with controlled return paths" (at 18 77) (layer "Cmts.User"))
+  (gr_text "Ground stitching fence along motor section boundary" (at 43 76) (layer "Cmts.User"))
   (gr_circle (center 4 4) (end 5.6 4) (layer "Edge.Cuts") (width 0.1) (fill none))
   (gr_circle (center 96 4) (end 97.6 4) (layer "Edge.Cuts") (width 0.1) (fill none))
